File: Schaltpläne/Empfangsseite/Empfangseinheit.sch (EAGLE design)
At the start: 25 parts, among them IC2 TL074P, X1 +5V,0V,-5V

Commit message: Schematics updated
Empfangseinheit baby
Parts:
- removed R_VOR_SENDE: 10, resistor:R-EU_0207_10
- added R_RECEIVER: 10, resistor:R-EU_0207_10
- added X2: (no value), con-phoenix-254:MPT2
- X1: value +5V,0V,-5V -> (none)
Connections:
- net N$5 renamed RAW_SIGNAL
- removed net N$10: IC2A.+IN, R12.2
- new net N$7: C7.2, IC2A.+IN, R12.2
- net FINAL_OUTPUT: now also R3.A, X2-1.1; no longer R3.E
- net FINAL_SIGNAL: now also R3.E; no longer R3.A
- net GND: now also X2-2.1; no longer C7.1, RECEIVER_DIODE.GND
- net N$9: now also R_RECEIVER.1; no longer R_VOR_SENDE.1
- net POST_FILTER: now also C7.1; no longer C7.2
- net V+: now also R_RECEIVER.2; no longer R_VOR_SENDE.2
Other:
- note added: "Dennis Ernst Clemens Büsch"
- note added: "Optische Übertragungsstrecke"
- note added: "Semesterprojekt"
- note removed: "Stütz TL074"
- moved on the sheet: C1, C2, C3, C4, C5, C6, C7, C9, DIODE, IC2A, IC2B, IC2C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
